Commit message: commit

File: urdf/puzzlebot_jetson_ed_urdf.urdf (robot description, URDF)
Before this commit: robot Puzzlebot Jetson-Lidar Ed., 2 links, 1 joints
Links:
- added link wheel1, mass 0.01; collision mesh filename=package://localisation/models/MCR2_1000_1_1_Wheel_Coupler_2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; visual mesh filename=package://localisation/models/MCR2_1000_1_1_Wheel_Coupler_2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
- added link wheel2, mass 0.01; collision mesh filename=package://localisation/models/MCR2_1000_1_1_Wheel_Coupler_2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; visual mesh filename=package://localisation/models/MCR2_1000_1_1_Wheel_Coupler_2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
Joints:
- added joint wheel_joint1: type continuous, parent chassis, child wheel1, origin xyz=0.3 0.15 0.0
- added joint wheel_joint2: type continuous, parent chassis, child wheel2, origin xyz=0.3 -0.15 0.0

Commit message: Update puzzlebot_jetson_ed_urdf.urdf

File: urdf/puzzlebot_jetson_ed_urdf.urdf (robot description, URDF)
Before this commit: robot Puzzlebot Jetson-Lidar Ed., 4 links, 3 joints
Joints:
- joint wheel_joint1: origin xyz=0.3 0.15 0.0 -> xyz=0.0 -0.15 0.0 rpy=0 0 1.5708
- joint wheel_joint2: origin xyz=0.3 -0.15 0.0 -> xyz=0.0 0.15 0.0 rpy=0 0 -1.5708

Commit message: webos_potter

File: urdf/puzzlebot_jetson_ed_urdf.urdf (robot description, URDF)
Before this commit: robot Puzzlebot Jetson-Lidar Ed., 4 links, 3 joints
Links:
- link chassis: geometry collision mesh filename=package://puzzlebot_sim/models/MCR2_1000_13_Chassis.stl; visual mesh filename=package://puzzlebot_sim/models/MCR2_1000_13_Chassis.stl
- link wheel1: geometry collision mesh filename=package://puzzlebot_sim/models/MCR2_1000_1_1_Wheel_Coupler_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; visual mesh filename=package://puzzlebot_sim/models/MCR2_1000_1_1_Wheel_Coupler_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
- link wheel2: geometry collision mesh filename=package://puzzlebot_sim/models/MCR2_1000_1_1_Wheel_Coupler_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; visual mesh filename=package://puzzlebot_sim/models/MCR2_1000_1_1_Wheel_Coupler_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

Commit message: puzzlebot_jetson_ed_urdf.urdf

File: urdf/puzzlebot_jetson_ed_urdf.urdf (robot description, URDF)
Before this commit: robot Puzzlebot Jetson-Lidar Ed., 4 links, 3 joints
Links:
- link chassis: geometry collision mesh filename=package://localisation/models/MCR2_1000_13_Chassis.stl; visual mesh filename=package://localisation/models/MCR2_1000_13_Chassis.stl
- link wheel1: geometry collision mesh filename=package://localisation/models/MCR2_1000_1_1_Wheel_Coupler_2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; visual mesh filename=package://localisation/models/MCR2_1000_1_1_Wheel_Coupler_2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
- link wheel2: geometry collision mesh filename=package://localisation/models/MCR2_1000_1_1_Wheel_Coupler_2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; visual mesh filename=package://localisation/models/MCR2_1000_1_1_Wheel_Coupler_2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
Joints:
- joint wheel_joint1: origin xyz=0.0 -0.15 0.0 rpy=0 0 1.5708 -> xyz=0.052 0.0972 0.0 rpy=1.5708 0 -1.5708
- joint wheel_joint2: origin xyz=0.0 0.15 0.0 rpy=0 0 -1.5708 -> xyz=0.052 -0.0972 0.0 rpy=-1.5708 0 1.5708

Commit message: commit

File: urdf/puzzlebot_jetson_ed_urdf.urdf (robot description, URDF)
Before this commit: robot Puzzlebot Jetson-Lidar Ed., 4 links, 3 joints
Joints:
- removed joint wheel_joint1
- removed joint wheel_joint2
- added joint joint_wheel1: type continuous, parent chassis, child wheel1, origin xyz=0.052 0.0972 0.0 rpy=1.5708 0 -1.5708
- added joint joint_wheel2: type continuous, parent chassis, child wheel2, origin xyz=0.052 -0.0972 0.0 rpy=-1.5708 0 1.5708

Commit message: commit

File: urdf/puzzlebot_jetson_ed_urdf.urdf (robot description, URDF)
Before this commit: robot Puzzlebot Jetson-Lidar Ed., 4 links, 3 joints
Joints:
- removed joint joint_wheel1
- removed joint joint_wheel2
- added joint wheel_joint1: type continuous, parent chassis, child wheel1, origin xyz=0.052 0.0972 0.0 rpy=1.5708 0 -1.5708
- added joint wheel_joint2: type continuous, parent chassis, child wheel2, origin xyz=0.052 -0.0972 0.0 rpy=-1.5708 0 1.5708

Commit message: commit

File: urdf/puzzlebot_jetson_ed_urdf.urdf (robot description, URDF)
Before this commit: robot Puzzlebot Jetson-Lidar Ed., 4 links, 3 joints
Joints:
- joint wheel_joint1: origin xyz=0.052 0.0972 0.0 rpy=1.5708 0 -1.5708 -> xyz=0.052 0.0972 0.0 rpy=-1.5708 0 1.5708
